Commit message: add distortion and fisheye model

File: franka_cal_sim/xacro/aprilgrid.xacro (robot description, xacro)
@@ -8,5 +8,5 @@
       <parent link="world"/>
       <child link="simple_box_base_link"/>
-      <origin rpy="0.0 1.5707 0" xyz="-2.0 -0.4 0.4"/>
+      <origin rpy="0.0 1.5707 0" xyz="-2.0 -0.35 0.5"/>
     </joint>
     <link name="simple_box_base_link">

File: franka_ros/franka_description/robots/hand.xacro (robot description, xacro)
@@ -72,5 +72,6 @@
       <parent link="${ns}_hand"/>
       <child link="${ns}_rightfinger"/>
-      <origin xyz="0 0 0.0584" rpy="0 0 0"/>
+<origin xyz="0.0037056166097622547 -0.010068426985226817 0.04390725799202158" rpy="0.016289975357708444 -0.2681597342670168 -0.14954467264378038"/>
+<!--y+0.01:x-0.01,x-0.01:y-0.01,z+0.01,z+0.01-->
       <axis xyz="0 -1 0"/>
       <limit effort="20" lower="0.03" upper="0.03" velocity="0.2"/>

File: franka_ros/franka_description/robots/panda.gazebo.xacro (robot description, xacro)
@@ -77,8 +77,8 @@
 	  <gazebo reference="${robot_name}_leftfinger">
 	    <sensor type="camera" name="camera">
-	      <update_rate>7.0</update_rate><!--20-->
+	      <update_rate>10</update_rate><!--10-->
 	      <camera name="camera">
-                <pose>0.0 0.0 0.1 0 -1.57 0</pose>
-		<horizontal_fov>1.0</horizontal_fov>
+                <pose>0.0 0.0 0.1 0 -1.5708 0</pose>
+<horizontal_fov>0.93137074148</horizontal_fov>
 		<image>
 		  <width>640</width>
@@ -88,6 +88,14 @@
 		<clip>
 		  <near>0.005</near>
-		  <far>4</far>
+		  <far>100</far>
 		</clip>
+                <distortion>
+            <k1>0.2</k1>
+            <k2>0.2</k2>
+            <k3>0.0</k3>
+            <p1>-0.0000</p1>
+            <p2>-0.0000</p2>
+            <center>0.5 0.5</center>
+          </distortion>
 		<noise>
 		  <type>gaussian</type>
@@ -95,17 +103,35 @@
 		  <stddev>0.0</stddev>
 		</noise>
+<lens>
+      <!-- type element is mandatory -->
+      <type>custom</type>
+      <!-- manually defined mapping function r = c1*f*fun(theta/c2 + c3) -->
+      <!-- More information here: https://en.wikipedia.org/wiki/Fisheye_lens#Mapping_function -->
+      <custom_function>
+        <c1>1.05</c1>
+        <!-- linear scaling -->
+        <c2>4</c2>
+        <!-- angle scaling -->
+        <f>1.0</f>
+        <!-- one more scaling parameter -->
+        <fun>tan</fun>
+        <!-- one of sin,tan,id -->
+      </custom_function>
+      <!-- if it is set to `true` your horizontal FOV will ramain as defined -->
+      <!-- othervise it depends on lens type and custom function, if there is one -->
+      <scale_to_hfov>true</scale_to_hfov>
+      <!-- clip everything that is outside of this angle -->
+      <cutoff_angle>3.1415</cutoff_angle>
+      <!-- resolution of the cubemap texture, the highter it is - the sharper is your image -->
+      <env_texture_size>512</env_texture_size>
+    </lens>
 	      </camera>
 	      <plugin name="camera_controller" filename="libgazebo_ros_camera.so">
 		<alwaysOn>true</alwaysOn>
-		<updateRate>0.0</updateRate>
 		<cameraName>simple_camera</cameraName>
 		<imageTopicName>image_raw</imageTopicName>
 		<cameraInfoTopicName>camera_info</cameraInfoTopicName>
 		<frameName>camera_link</frameName>
-		<distortionK1>0.0</distortionK1>
-		<distortionK2>0.0</distortionK2>
-		<distortionK3>0.0</distortionK3>
-		<distortionT1>0.0</distortionT1>
-		<distortionT2>0.0</distortionT2>
+                <hackBaseline>0.0</hackBaseline>
 	      </plugin>
 	    </sensor>
@@ -120,12 +146,12 @@
 	  <serviceName>/imu/service</serviceName>
 	  <accelOffset>0 0 0</accelOffset>
-	  <accelDrift>0.006 0.006 0.006</accelDrift>
-	  <accelGaussianNoise>0.004 0.004 0.004</accelGaussianNoise>
+	  <accelDrift>0.006 0.006 0.006</accelDrift><!--0.006-->
+	  <accelGaussianNoise>0.004 0.004 0.004</accelGaussianNoise><!--0.004-->
 	  <rateDrift>0.000038785 0.000038785 0.000038785</rateDrift>
 	  <rateGaussianNoise>0.0003394 0.0003394 0.0003394</rateGaussianNoise>
 	  <yawOffset>0.0 0.0 0.0</yawOffset>
-	  <yawDrift>0.000038785 0.000038785 0.000038785</yawDrift>
+	  <yawDrift>0.0 0.0 0.0</yawDrift>
 	  <yawDriftFrequency>0.0 0.0 0.0</yawDriftFrequency>
-	  <yawGaussianNoise>0.0003394 0.0003394 0.0003394</yawGaussianNoise>
+	  <yawGaussianNoise>0.0 0.0 0.0</yawGaussianNoise>
 	  <gaussianNoise>0.0</gaussianNoise>
 	</plugin>

File: franka_ros/franka_description/robots/panda_arm.xacro (robot description, xacro)
@@ -53,9 +53,9 @@
     <joint name="${arm_id}_joint1" type="revolute">
       <safety_controller k_position="100.0" k_velocity="40.0" soft_lower_limit="-2.8973" soft_upper_limit="2.8973"/>
-      <origin rpy="0 0 0" xyz="0 0 0.333"/>
+      <origin rpy="0 0 0.0" xyz="0 0 0.333"/>
       <parent link="${arm_id}_link0"/>
       <child link="${arm_id}_link1"/>
       <axis xyz="0 0 1"/>
-      <limit effort="87" lower="-2.8973" upper="2.8973" velocity="2.1750"/>
+      <limit effort="87" lower="-2.8973" upper="2.8973" velocity="2.1750"/> <!--effort 87-->
       <dynamics damping="${joint_damping}"/>
     </joint>
@@ -79,9 +79,9 @@
     <joint name="${arm_id}_joint2" type="revolute">
       <safety_controller k_position="100.0" k_velocity="40.0" soft_lower_limit="-1.7628" soft_upper_limit="1.7628"/>
-      <origin rpy="${-pi/2} 0 0" xyz="0 0 0"/>
+      <origin rpy="${-pi/2} 0 0" xyz="0 0 0"/><!--(0)-->
       <parent link="${arm_id}_link1"/>
       <child link="${arm_id}_link2"/>
       <axis xyz="0 0 1"/>
-      <limit effort="87" lower="-1.7628" upper="1.7628" velocity="2.1750"/>
+      <limit effort="87" lower="-1.7628" upper="1.7628" velocity="2.1750"/> <!--effort 87-->
       <dynamics damping="${joint_damping}"/>
     </joint>
@@ -105,9 +105,9 @@
     <joint name="${arm_id}_joint3" type="revolute">
       <safety_controller k_position="100.0" k_velocity="40.0" soft_lower_limit="-2.8973" soft_upper_limit="2.8973"/>
-      <origin rpy="${pi/2} 0 0" xyz="0 -0.316 0"/>
+      <origin rpy="${pi/2} 0 0" xyz="0 -0.316 0"/><!--r=pi/2-->
       <parent link="${arm_id}_link2"/>
       <child link="${arm_id}_link3"/>
       <axis xyz="0 0 1"/>
-      <limit effort="87" lower="-2.8973" upper="2.8973" velocity="2.1750"/>
+      <limit effort="87" lower="-2.8973" upper="2.8973" velocity="2.1750"/> <!--effort 87-->
       <dynamics damping="${joint_damping}"/>
     </joint>
@@ -131,9 +131,9 @@
     <joint name="${arm_id}_joint4" type="revolute">
       <safety_controller k_position="100.0" k_velocity="40.0" soft_lower_limit="-3.0718" soft_upper_limit="-0.0698"/>
-      <origin rpy="${pi/2} 0 0" xyz="0.0825 0 0"/>
+      <origin rpy="${pi/2} 1.0 0" xyz="0.0825 0 0"/> <!--0 p=${pi/4}-->
       <parent link="${arm_id}_link3"/>
       <child link="${arm_id}_link4"/>
       <axis xyz="0 0 1"/>
-      <limit effort="87" lower="-3.0718" upper="-0.0698" velocity="2.1750"/>
+      <limit effort="87" lower="-3.0718" upper="-0.0698" velocity="2.1750"/> <!--effort 87-->
       <dynamics damping="${joint_damping}"/>
     </joint>
@@ -183,5 +183,5 @@
     <joint name="${arm_id}_joint6" type="revolute">
       <safety_controller k_position="100.0" k_velocity="40.0" soft_lower_limit="-0.0175" soft_upper_limit="3.7525"/>
-      <origin rpy="${pi/2} 0 0" xyz="0 0 0"/>
+      <origin rpy="${pi/2} -${pi/2} 0" xyz="0 0 0"/> <!--p==0--><!---pi/2-->
       <parent link="${arm_id}_link5"/>
       <child link="${arm_id}_link6"/>

File: franka_ros/franka_description/robots/panda_arm_hand.urdf.xacro (robot description, xacro)
@@ -9,4 +9,4 @@
   <xacro:hand ns="panda" rpy="0 0 ${-pi/4}" connected_to="panda_link8"/>
   <xacro:panda_gazebo robot_name="$(arg robot_name)" />
-  <xacro:panda_transmission robot_name="$(arg robot_name)" />
+  <xacro:panda_transmission robot_name="$(arg robot_name)"/>
 </robot>
