Commit message: add randomness for distortion

File: franka_ros/franka_description/robots/hand.xacro (robot description, xacro)
@@ -72,5 +72,5 @@
       <parent link="${ns}_hand"/>
       <child link="${ns}_rightfinger"/>
-<origin xyz="0.0037056166097622547 -0.010068426985226817 0.04390725799202158" rpy="0.016289975357708444 -0.2681597342670168 -0.14954467264378038"/>
+<origin xyz="0.013837671108054209 -0.0290349966794423 0.07272135655650828" rpy="0.13281813239921123 0.15522038604111385 -0.008245936800331618"/>
 <!--y+0.01:x-0.01,x-0.01:y-0.01,z+0.01,z+0.01-->
       <axis xyz="0 -1 0"/>

File: franka_ros/franka_description/robots/panda.gazebo.xacro (robot description, xacro)
@@ -80,5 +80,5 @@
 	      <camera name="camera">
                 <pose>0.0 0.0 0.1 0 -1.5708 0</pose>
-<horizontal_fov>0.93137074148</horizontal_fov>
+<horizontal_fov>1.00669419933</horizontal_fov>
 		<image>
 		  <width>640</width>
@@ -91,9 +91,9 @@
 		</clip>
                 <distortion>
-            <k1>0.2</k1>
-            <k2>0.2</k2>
-            <k3>0.0</k3>
-            <p1>-0.0000</p1>
-            <p2>-0.0000</p2>
+<k1>0.23867294373626566</k1>
+<k2>0.69533407092404</k1>
+<k3>-0.0976259174516057</k1>
+<p1>-0.0000</p1>
+<p2>-0.0000</p2>
             <center>0.5 0.5</center>
           </distortion>
